Commit message: connected ros2 controller

File: urdf/2d_lidar/sick_s300.urdf.xacro (robot description, xacro)
@@ -12,5 +12,4 @@
                        topic_prefix:=~/
                        gpu:=false">
-    <!-- node_namespace is used from node_name if not set -->
     <xacro:if value="${node_namespace == None}">
       <xacro:property name="node_namespace" value="${frame_prefix}"/>

File: urdf/all_sensors.urdf.xacro (robot description, xacro)
@@ -1,47 +1,7 @@
 <?xml version="1.0"?>
 <robot name="all_sensors" xmlns:xacro="http://wiki.ros.org/xacro">
-  <!-- This file unifies all sensors that can be used on simulation, defined as xacro:macros -->
   <xacro:include filename="$(find golf_cart)/urdf/utils/inertia.urdf.xacro" />
-  <!-- Depth sensors -->
-  <!-- <xacro:include filename="$(find golf_cart)/urdf/depth/intel_realsense_d435.urdf.xacro" />
-  <xacro:include filename="$(find golf_cart)/urdf/depth/intel_realsense_d435i.urdf.xacro" /> -->
   <xacro:include filename="$(find golf_cart)/urdf/depth/orbbec_astra.urdf.xacro" />
-  <!-- <xacro:include filename="$(find golf_cart)/urdf/depth/stereolabs_generic.urdf.xacro" />
-  <xacro:include filename="$(find golf_cart)/urdf/depth/stereolabs_zed2.urdf.xacro" />
-  <xacro:include filename="$(find golf_cart)/urdf/depth/stereolabs_zed2i.urdf.xacro" />
-  <xacro:include filename="$(find golf_cart)/urdf/depth/azure_kinect.urdf.xacro" /> -->
-  <!-- 2D Lidars -->
-  <!-- <xacro:include filename="$(find golf_cart)/urdf/2d_lidar/sick_microscan3.urdf.xacro" />
-  <xacro:include filename="$(find golf_cart)/urdf/2d_lidar/sick_nanoscan3.urdf.xacro" />
-  <xacro:include filename="$(find golf_cart)/urdf/2d_lidar/sick_outdoorscan3.urdf.xacro" /> -->
   <xacro:include filename="$(find golf_cart)/urdf/2d_lidar/sick_s300.urdf.xacro" />
-  <!-- <xacro:include filename="$(find golf_cart)/urdf/2d_lidar/sick_s3000.urdf.xacro" />
-  <xacro:include filename="$(find golf_cart)/urdf/2d_lidar/sick_tim551.urdf.xacro" />
-  <xacro:include filename="$(find golf_cart)/urdf/2d_lidar/sick_tim571.urdf.xacro" />
-  <xacro:include filename="$(find golf_cart)/urdf/2d_lidar/hokuyo_urg04lx.urdf.xacro" />
-  <xacro:include filename="$(find golf_cart)/urdf/2d_lidar/hokuyo_ust10lx.urdf.xacro" />
-  <xacro:include filename="$(find golf_cart)/urdf/2d_lidar/hokuyo_ust20lx.urdf.xacro" />
-  <xacro:include filename="$(find golf_cart)/urdf/2d_lidar/hokuyo_utm30lx.urdf.xacro" /> -->
-  <!-- 3D Lidars -->
-  <!-- <xacro:include filename="$(find golf_cart)/urdf/3d_lidar/velodyne_vlp16.urdf.xacro" />
-  <xacro:include filename="$(find golf_cart)/urdf/3d_lidar/robosense_bpearl.urdf.xacro" />
-  <xacro:include filename="$(find golf_cart)/urdf/3d_lidar/robosense_helios_16p.urdf.xacro" />
-  <xacro:include filename="$(find golf_cart)/urdf/3d_lidar/ouster.urdf.xacro" />
-  <xacro:include filename="$(find golf_cart)/urdf/3d_lidar/livox_mid_360.urdf.xacro" />
-  <xacro:include filename="$(find golf_cart)/urdf/3d_lidar/sick_multiscan_100.urdf.xacro" /> -->
-  <!-- IMUs -->
-  <!-- <xacro:include filename="$(find golf_cart)/urdf/imu/vectornav.urdf.xacro" /> -->
   <xacro:include filename="$(find golf_cart)/urdf/imu/myahrs.urdf.xacro" />
-  <!-- <xacro:include filename="$(find golf_cart)/urdf/imu/pixhawk.urdf.xacro" /> -->
-  <!-- GPS -->
-  <!-- <xacro:include filename="$(find golf_cart)/urdf/gps/gps.urdf.xacro" />
-  <xacro:include filename="$(find golf_cart)/urdf/gps/gps_with_mast.urdf.xacro" />
-  <xacro:include filename="$(find golf_cart)/urdf/gps/ublox.urdf.xacro" />
-  <xacro:include filename="$(find golf_cart)/urdf/gps/ublox_with_mast.urdf.xacro" /> -->
-  <!-- Camera -->
-  <!-- <xacro:include filename="$(find golf_cart)/urdf/camera/axis_m5013.urdf.xacro" />
-  <xacro:include filename="$(find golf_cart)/urdf/camera/axis_m5074.urdf.xacro" />
-  <xacro:include filename="$(find golf_cart)/urdf/camera/axis_m5525.urdf.xacro" />
-  <xacro:include filename="$(find golf_cart)/urdf/camera/axis_m5526.urdf.xacro" />
- -->
 </robot>

File: urdf/depth/orbbec_astra.urdf.xacro (robot description, xacro)
@@ -11,5 +11,4 @@
                        node_name:=orbbec_astra
                        topic_prefix:=~/">
-    <!-- node_namespace is used from node_name if not set -->
     <xacro:if value="${node_namespace == None}">
       <xacro:property name="node_namespace" value="${node_name}"/>

File: urdf/imu/imu_plugin.urdf.xacro (robot description, xacro)
@@ -21,5 +21,4 @@
                 <noise type="gaussian">
                   <mean>0.0</mean>
-                  <!-- <stddev>2e-3</stddev> -->
                   <stddev>0.01</stddev>
                 </noise>
@@ -28,5 +27,4 @@
                 <noise type="gaussian">
                   <mean>0.0</mean>
-                  <!-- <stddev>2e-3</stddev> -->
                   <stddev>0.01</stddev>
                 </noise>
@@ -35,5 +33,4 @@
                 <noise type="gaussian">
                   <mean>0.0</mean>
-                  <!-- <stddev>2e-3</stddev> -->
                   <stddev>0.01</stddev>
                 </noise>
@@ -44,5 +41,4 @@
                 <noise type="gaussian">
                   <mean>0.0</mean>
-                  <!-- <stddev>2e-4</stddev> -->
                   <stddev>0.01</stddev>
                 </noise>
@@ -51,5 +47,4 @@
                 <noise type="gaussian">
                   <mean>0.0</mean>
-                  <!-- <stddev>2e-4</stddev> -->
                   <stddev>0.01</stddev>
                 </noise>
@@ -58,5 +53,4 @@
                 <noise type="gaussian">
                   <mean>0.0</mean>
-                  <!-- <stddev>2e-3</stddev> -->
                   <stddev>0.01</stddev>
                 </noise>
@@ -67,5 +61,4 @@
                 <noise type="gaussian">
                   <mean>0.0</mean>
-                  <!-- <stddev>1.7e-2</stddev> -->
                   <stddev>0.01</stddev>
                 </noise>
@@ -74,5 +67,4 @@
                 <noise type="gaussian">
                   <mean>0.0</mean>
-                  <!-- <stddev>1.7e-2</stddev> -->
                   <stddev>0.01</stddev>
                 </noise>
@@ -81,5 +73,4 @@
                 <noise type="gaussian">
                   <mean>0.0</mean>
-                  <!-- <stddev>1.7e-2</stddev> -->
                   <stddev>0.01</stddev>
                 </noise>

File: urdf/inertia.urdf.xacro (robot description, xacro)
@@ -1,6 +1,4 @@
 <?xml version="1.0"?>
 <robot xmlns:xacro="http://www.ros.org/wiki/xacro">
-  <!-- Source: https://en.wikipedia.org/wiki/List_of_moments_of_inertia-->
-  <!-- Solid sphere of radius r and mass m-->
   <xacro:macro name="solid_sphere_inertia" params="m r">
     <inertia  ixx="${(2*r*r*m)/5}" ixy = "0" ixz = "0"
@@ -9,5 +7,4 @@
     />
   </xacro:macro>
-  <!-- Hollow sphere of radius r and mass m-->
   <xacro:macro name="solid_sphere_inertia" params="m r">
     <inertia  ixx="${(2*r*r*m)/3}" ixy = "0" ixz = "0"
@@ -16,5 +13,4 @@
     />
   </xacro:macro>
-  <!-- Solid ellipsoid of semi-axes a, b, c and mass m-->
   <xacro:macro name="ellipsoid_semi_axes_inertia" params="a b c m r">
     <inertia  ixx="${(m*(b*b+c*c))/5}" ixy = "0" ixz = "0"
@@ -23,5 +19,4 @@
     />
   </xacro:macro>
-  <!-- Right circular cone with radius r, height h and mass m, about the apex -->
   <xacro:macro name="right_circular_cone_inertia" params="m r h">
     <inertia  ixx="${((3*m*(h*h))/5)+((3*m*(r*r))/20)}" ixy = "0" ixz = "0"
@@ -30,5 +25,4 @@
     />
   </xacro:macro>
-  <!-- Solid cuboid of width w, height h, depth d, and mass m -->
   <xacro:macro name="solid_cuboid_inertia" params="m h d w">
     <inertia  ixx="${(m*(h*h+d*d))/12}" ixy = "0" ixz = "0"
@@ -37,5 +31,4 @@
     />
   </xacro:macro>
-  <!-- Solid cylinder of radius r, height h and mass m -->
   <xacro:macro name="solid_cylinder_inertia" params="m r h">
     <inertia  ixx="${m*(3*r*r+h*h)/12}" ixy = "0" ixz = "0"
@@ -44,5 +37,4 @@
     />
   </xacro:macro>
-  <!-- Thick-walled cylindrical tube with open ends, of inner radius r1, outer radius r2, length h and mass m -->
   <xacro:macro name="thick_walled_cylinder_inertia" params="m r1 r2 h">
     <inertia  ixx="${m*((3*(r1*r1+r2*r2))+(h*h))/12}" ixy = "0" ixz = "0"

File: urdf/ros2_control.urdf.xacro (robot description, xacro)
@@ -14,5 +14,4 @@
           <state_interface name="velocity"/>
           <state_interface name="position"/>
-          <!-- <state_interface name="effort"/> -->
         </joint>
         <joint name="summit_xl_front_right_wheel_joint">
@@ -23,5 +22,4 @@
           <state_interface name="velocity"/>
           <state_interface name="position"/>
-          <!-- <state_interface name="effort"/> -->
         </joint>
         <joint name="summit_xl_back_left_wheel_joint">
@@ -32,5 +30,4 @@
           <state_interface name="velocity"/>
           <state_interface name="position"/>
-          <!-- <state_interface name="effort"/> -->
         </joint>
         <joint name="summit_xl_back_right_wheel_joint">
@@ -41,14 +38,6 @@
           <state_interface name="velocity"/>
           <state_interface name="position"/>
-          <!-- <state_interface name="effort"/> -->
         </joint>
       </ros2_control>
-      <!-- <gazebo>
-        <plugin name="gazebo_ros2_control" filename="libgazebo_ros2_control.so">
-          <namespace>$(arg robot_id)</namespace>
-          <parameters>$(arg config_controllers)</parameters>
-          <parameters>$(find golf_cart)/config/simulation/ros2_control.yaml</parameters>
-        </plugin>
-      </gazebo> -->
       <gazebo>
         <plugin name="gazebo_ros2_control" filename="libgazebo_ros2_control.so">

File: urdf/summit_xls.urdf.xacro (robot description, xacro)
@@ -1,21 +1,12 @@
 <?xml version="1.0"?>
 <robot name="summit_xl" xmlns:xacro="http://wiki.ros.org/xacro">
-	<!-- ***************** -->
-	<!-- Imported elements -->
-	<!-- ***************** -->
-	<!-- First we import all posible elements defined in the urdf.xacro files. All these elements are defined as macro:xacros -->
-	<!-- Import summit XL base elements -->
 	<xacro:include filename="$(find golf_cart)/urdf/summit_xls_base.urdf.xacro" />
 	<xacro:include filename="$(find golf_cart)/urdf/ros2_control.urdf.xacro" />
-	<!-- Import summit XL wheels -->
 	<xacro:include filename="$(find golf_cart)/urdf/wheels/omni_wheel.urdf.xacro" />
 	<xacro:include filename="$(find golf_cart)/urdf/wheels/rubber_wheel.urdf.xacro" />
 	<xacro:include filename="$(find golf_cart)/urdf/structures/structure_hokuyo.urdf.xacro" />
-	<!-- Import all available sensors -->
 	<xacro:include filename="$(find golf_cart)/urdf/all_sensors.urdf.xacro" />
 	<xacro:property name="PI" value="3.1415926535897931"/>
-	<!-- Wheel parameters -->
-	<!-- Wheel parameters -->
-	<xacro:property name="wheel_offset_x" value="0.2225" />    <!-- x,y,z in translation from base_link to the center of the wheel -->
+	<xacro:property name="wheel_offset_x" value="0.2225" />
 	<xacro:property name="wheel_offset_y" value="0.2045" />
 	<xacro:property name="wheel_offset_z" value="0.0" />
@@ -41,51 +32,34 @@
 	<xacro:property name="gps_offset_y" value="-0.167"/>
 	<xacro:property name="gps_offset_z" value="0.302"/>
-	<!-- Flag to select the high or low quality model -->
 	<xacro:property name="hq" value="false" />
 	<xacro:arg name="prefix" default="summit_xl_"/>
-	<xacro:arg name="ros_planar_move_plugin" default="false"/>
+	<xacro:arg name="ros_planar_move_plugin" default="true"/>
 	<xacro:arg name="gpu" default="false"/>
     <xacro:macro name="summit_xl" params="prefix publish_bf hq">
-		<!-- *************** -->
-		<!-- Robots Elements -->
-		<!-- *************** -->
-		<!-- Here we create the robot elements using the xacro:macros imported at the beggining of this file -->
-		<!-- Summit XL base -->
 		<xacro:summit_xls_base prefix="$(arg prefix)" publish_bf="true" hq="${hq}" />
-		<xacro:omni_wheel prefix="$(arg prefix)front_right" parent="$(arg prefix)base_link" reflect="false" hq="${hq}">
+		<xacro:rubber_wheel prefix="$(arg prefix)front_right" parent="$(arg prefix)base_link" reflect="false" hq="${hq}">
 			<origin xyz="${wheel_offset_x} -${wheel_offset_y} ${wheel_offset_z}" rpy="0 0 0"/>
-		</xacro:omni_wheel>
-		<xacro:omni_wheel prefix="$(arg prefix)front_left" parent="$(arg prefix)base_link" reflect="true" hq="${hq}">
+		</xacro:rubber_wheel>
+		<xacro:rubber_wheel prefix="$(arg prefix)front_left" parent="$(arg prefix)base_link" reflect="true" hq="${hq}">
 			<origin xyz="${wheel_offset_x} ${wheel_offset_y} ${wheel_offset_z}" rpy="0 0 0"/>
-		</xacro:omni_wheel>
-		<xacro:omni_wheel prefix="$(arg prefix)back_left" parent="$(arg prefix)base_link" reflect="true" hq="${hq}">
+		</xacro:rubber_wheel>
+		<xacro:rubber_wheel prefix="$(arg prefix)back_left" parent="$(arg prefix)base_link" reflect="true" hq="${hq}">
 			<origin xyz="-${wheel_offset_x} ${wheel_offset_y} ${wheel_offset_z}" rpy="0 0 0"/>
-		</xacro:omni_wheel>
-		<xacro:omni_wheel prefix="$(arg prefix)back_right" parent="$(arg prefix)base_link" reflect="false" hq="${hq}">
+		</xacro:rubber_wheel>
+		<xacro:rubber_wheel prefix="$(arg prefix)back_right" parent="$(arg prefix)base_link" reflect="false" hq="${hq}">
 			<origin xyz="-${wheel_offset_x} -${wheel_offset_y} ${wheel_offset_z}" rpy="0 0 0"/>
-		</xacro:omni_wheel>
-        <!-- IMU -->
+		</xacro:rubber_wheel>
 		<xacro:sensor_myahrs frame_prefix="$(arg prefix)imu" parent="$(arg prefix)base_link">
 			<origin xyz="${imu_offset_x} ${imu_offset_y} ${imu_offset_z}" rpy="0 0 0"/>
 		</xacro:sensor_myahrs>
-		<!-- SENSORS -->
-		<xacro:sensor_sick_s300 frame_prefix="$(arg prefix)front_laser" parent="$(arg prefix)base_link" topic_prefix="front_laser" gpu="$(arg gpu)">
+		<xacro:sensor_orbbec_astra frame_prefix="$(arg prefix)front_rgbd_camera" parent="$(arg prefix)base_link" topic_prefix="front_rgbd_camera">
+			<origin xyz="${front_rgbd_camera_offset_x} ${front_rgbd_camera_offset_y} ${front_rgbd_camera_offset_z}" rpy="0 0 0"/>
+		</xacro:sensor_orbbec_astra>
+		<!-- <xacro:sensor_sick_s300 frame_prefix="$(arg prefix)front_laser" parent="$(arg prefix)base_link" topic_prefix="front_laser" gpu="$(arg gpu)">
 			<origin xyz="${front_laser_offset_x} ${front_laser_offset_y} ${front_laser_offset_z}" rpy="0 ${-PI} ${3/4*PI}" />
 		</xacro:sensor_sick_s300>
 		<xacro:sensor_sick_s300 frame_prefix="$(arg prefix)rear_laser" parent="$(arg prefix)base_link" topic_prefix="rear_laser" gpu="$(arg gpu)">
 			<origin xyz="${rear_laser_offset_x} ${rear_laser_offset_y} ${rear_laser_offset_z}" rpy="0 ${-PI} ${-1/4*PI}" />
-		</xacro:sensor_sick_s300>
-		<!--xacro:sensor_axis_m5013 prefix="$(arg prefix)front_ptz_camera" parent="$(arg prefix)base_link">
-			<origin xyz="${front_ptz_camera_offset_x} ${front_ptz_camera_offset_y} ${front_ptz_camera_offset_z}" rpy="${-PI/2} 0 0"/>
-		</xacro:sensor_axis_m5013-->
-		<!--xacro:sensor_axis_m5013 prefix="$(arg prefix)rear_ptz_camera" parent="$(arg prefix)base_link">
-			<origin xyz="${rear_ptz_camera_offset_x} ${rear_ptz_camera_offset_y} ${rear_ptz_camera_offset_z}" rpy="${-PI/2} 0 ${PI}"/>
-		</xacro:sensor_axis_m5013-->
-		<xacro:sensor_orbbec_astra frame_prefix="$(arg prefix)front_rgbd_camera" parent="$(arg prefix)base_link" topic_prefix="front_rgbd_camera">
-			<origin xyz="${front_rgbd_camera_offset_x} ${front_rgbd_camera_offset_y} ${front_rgbd_camera_offset_z}" rpy="0 0 0"/>
-		</xacro:sensor_orbbec_astra>
-		<!--xacro:sensor_gps prefix="$(arg prefix)gps" parent="$(arg prefix)base_link">
-			<origin xyz="${gps_offset_x} ${gps_offset_y} ${gps_offset_z}" rpy="0 0 0"/>
-		</xacro:sensor_gps-->
+		</xacro:sensor_sick_s300> -->
    </xacro:macro>
    <xacro:ros2_control prefix="$(arg prefix)"/>
@@ -93,4 +67,4 @@
 	   <xacro:omni_steering prefix="$(arg prefix)" publish_tf="true"/>
    </xacro:if>
-   <xacro:summit_xl prefix="$(arg prefix)" publish_bf="true" hq="false"/>
+   <xacro:summit_xl prefix="$(arg prefix)" publish_bf="true" hq="${hq}"/>
 </robot>

File: urdf/summit_xls_base.urdf.xacro (robot description, xacro)
@@ -1,10 +1,7 @@
 <?xml version="1.0"?>
 <robot name="summit_xl" xmlns:xacro="http://wiki.ros.org/xacro">
-  <!-- <xacro:include filename="$(find golf_cart)/urdf/summit_xl_base.gazebo.xacro" /> -->
   <xacro:macro name="summit_xls_base" params="prefix publish_bf hq">
-  <!-- Robot mechanical and motor parameters -->
   <xacro:property name="PI" value="3.1415926535897931"/>
   <xacro:property name="wheel_radius" value="0.127" />
-	<!-- BASE FOOTPRINT -->
 	  <xacro:if value="${publish_bf}">
 		<link name="${prefix}base_footprint">
@@ -17,10 +14,9 @@
 		</link>
 		<joint name="${prefix}base_footprint_joint" type="fixed">
-		  <origin xyz="0 0 ${wheel_radius}" rpy="0 0 0" /> <!-- ${wheel_radius} property must be defined inside wheel description -->
+		  <origin xyz="0 0 ${wheel_radius}" rpy="0 0 0" />
 		  <parent link="${prefix}base_footprint"/>
 		  <child link="${prefix}base_link" />
 		</joint>
 	  </xacro:if>
-  <!-- BASE_LINK -->
   <link name="${prefix}base_link">
     <inertial>
@@ -55,11 +51,4 @@
     <material>Gazebo/Black</material>
   </gazebo>
-  <link name="${prefix}base_docking_contact">
-  </link>
-  <joint name="${prefix}base_docking_joint" type="fixed">
-    <origin xyz="0.35 0 0.09" rpy="0 0 0" />
-    <parent link="${prefix}base_link"/>
-    <child link="${prefix}base_docking_contact" />
-  </joint>
   </xacro:macro>
 </robot>

File: urdf/utils/inertia.urdf.xacro (robot description, xacro)
@@ -1,6 +1,4 @@
 <?xml version="1.0"?>
 <robot xmlns:xacro="http://wiki.ros.org/xacro">
-  <!-- source en.wikipedia.org/wiki/List_of_moments_of_inertia-->
-  <!-- TODO Solid sphere of radius r and mass m-->
   <xacro:macro name="solid_sphere_inertia" params="m r">
     <inertia  ixx="${(2*r*r*m)/5}" ixy = "0" ixz = "0"
@@ -9,5 +7,4 @@
      />
   </xacro:macro>
-  <!-- TODO Hollow sphere of radius r and mass m-->
   <xacro:macro name="solid_sphere_inertia" params="m r">
     <inertia  ixx="${(2*r*r*m)/3}" ixy = "0" ixz = "0"
@@ -16,5 +13,4 @@
      />
   </xacro:macro>
-  <!-- TODO Solid ellipsoid of semi-axes a, b, c and mass m-->
   <xacro:macro name="ellipsoid_semi_axes_inertia" params="a b c m r">
     <inertia  ixx="${(m*(b*b+c*c))/5}" ixy = "0" ixz = "0"
@@ -23,5 +19,4 @@
      />
   </xacro:macro>
-  <!-- TODO Right circular cone with radius r, height h and mass m, about the apex -->
   <xacro:macro name="right_circular_cone_inertia" params="m r h">
     <inertia  ixx="${((3*m*(h*h))/5)+((3*m*(r*r))/20)}" ixy = "0" ixz = "0"
@@ -30,7 +25,4 @@
      />
   </xacro:macro>
-  <!-- TODO Solid cuboid of width w, height h, depth d, and mass m -->
-  <!-- w relates to X axis, d to Z axis, and h to Y axis -->
-  <!-- Keep this comment -->
   <xacro:macro name="solid_cuboid_inertia" params="m w h d">
     <inertia  ixx="${(m*(h*h+d*d))/12}" ixy = "0" ixz = "0"
@@ -39,5 +31,4 @@
      />
   </xacro:macro>
-  <!-- TODO Solid cylinder of radius r, height h and mass m -->
   <xacro:macro name="solid_cylinder_inertia" params="m r h">
     <inertia  ixx="${m*(3*r*r+h*h)/12}" ixy = "0" ixz = "0"
@@ -46,5 +37,4 @@
      />
   </xacro:macro>
-    <!-- TODO Thick-walled cylindrical tube with open ends, of inner radius r1, outer radius r2, length h and mass m -->
     <xacro:macro name="thick_walled_cylinder_inertia" params="m r1 r2 h">
     <inertia  ixx="${m*((3*(r1*r1+r2*r2))+(h*h))/12}" ixy = "0" ixz = "0"

File: urdf/wheels/omni_wheel.urdf.xacro (robot description, xacro)
@@ -5,5 +5,5 @@
   <xacro:property name="omni_wheel_radius" value="0.127" />
   <xacro:property name="omni_wheel_height" value="0.087" />
-  <xacro:property name="omni_wheel_mass" value="6.5" /> <!-- in kg-->
+  <xacro:property name="omni_wheel_mass" value="6.5" />
   <xacro:macro name="cylinder_inertia" params="m r h">
     <inertia  ixx="${m*(3*r*r+h*h)/12}" ixy = "0" ixz = "0"
@@ -48,15 +48,5 @@
 				<origin xyz="0 0 0" rpy="${PI/2} 0 0" />
         <geometry>
-          <!--sphere radius="${omni_wheel_radius}" /-->
-<!--
-          <xacro:if value="${reflect}">
-              <mesh filename="file://$(find golf_cart)/meshes/wheels/omni_wheel_1.dae" />
-          </xacro:if>
-          <xacro:unless value="${reflect}">
-              <mesh filename="file://$(find golf_cart)/meshes/wheels/omni_wheel_2.dae" />
-					</xacro:unless>
--->
 					<cylinder length="${omni_wheel_height}" radius="${omni_wheel_radius}" />
-					<!-- sphere radius="${omni_wheel_radius}"/-->
         </geometry>
       </collision>
@@ -67,5 +57,4 @@
       </inertial>
     </link>
-    <!-- Transmission is important to link the joints and the controller (see summit_xl_control/config/summit_xl_control.yaml)-->
     <transmission name="${prefix}_wheel_joint_trans">
       <type>transmission_interface/SimpleTransmission</type>

File: urdf/wheels/rubber_wheel.urdf.xacro (robot description, xacro)
@@ -2,23 +2,19 @@
 <robot name="wheel" xmlns:xacro="http://wiki.ros.org/xacro">
   <xacro:include filename="$(find golf_cart)/urdf/inertia.urdf.xacro"/>
-  <!-- CONSTANTS -->
   <xacro:property name="M_PI" value="3.1415926535897931"/>
   <xacro:property name="rubber_wheel_radius" value="0.11"/>
   <xacro:property name="rubber_wheel_height" value="0.15"/>
   <xacro:property name="rubber_wheel_mass" value="6.5"/>
-  <!-- WHEEL XACRO -->
   <xacro:macro name="rubber_wheel" params="prefix parent *origin reflect hq">
-    <!--TIRE -->
-    <joint name="${prefix}wheel_joint" type="continuous">
+    <joint name="${prefix}_wheel_joint" type="continuous">
       <xacro:insert_block name="origin" />
       <parent link="${parent}"/>
-      <child link="${prefix}wheel_link"/>
+      <child link="${prefix}_wheel_link"/>
       <axis xyz="0 1 0" rpy="0 0 0" />
       <limit effort="100" velocity="100"/>
       <dynamics damping="0.05" friction="0.1"/>
     </joint>
-    <link name="${prefix}wheel_link">
+    <link name="${prefix}_wheel_link">
       <visual>
-        <!-- HIGH RESOLUTION WHEELS -->
         <xacro:if value="${hq}">
           <origin xyz="0 0 0" rpy="0 0 0" />
@@ -32,5 +28,4 @@
           </geometry>
         </xacro:if>
-       <!-- LOW RESOLUTION WHEELS -->
         <xacro:unless value="${hq}">
           <origin xyz="0 0 0" rpy="${M_PI/2} 0 0" />
@@ -52,5 +47,5 @@
       </inertial>
     </link>
-    <gazebo reference="${prefix}wheel_link">
+    <gazebo reference="${prefix}_wheel_link">
       <mu1>0.95</mu1>
       <mu2>0.90</mu2>
