Commit message: fixed all sensors and ros2_control load error

File: urdf/2d_lidar/sick_s300.urdf.xacro (robot description, xacro)
@@ -24,5 +24,5 @@
         <origin xyz="0 0 0" rpy="${-pi/2} 0 0"/>
         <geometry>
-          <mesh filename="package://golf_cart/meshes/2d_lidar/s300.dae"/>
+          <mesh filename="file://$(find golf_cart)/meshes/2d_lidar/s300.dae"/>
         </geometry>
       </visual>
@@ -30,5 +30,5 @@
         <origin xyz="0 0 0" rpy="${-pi/2} 0 0"/>
         <geometry>
-          <mesh filename="package://golf_cart/meshes/2d_lidar/s300.dae"/>
+          <mesh filename="file://$(find golf_cart)/meshes/2d_lidar/s300.dae"/>
         </geometry>
       </collision>

File: urdf/depth/orbbec_astra.urdf.xacro (robot description, xacro)
@@ -23,5 +23,5 @@
         <origin xyz="0 0 0" rpy="0 0 0"/>
         <geometry>
-          <mesh filename="package://golf_cart/meshes/depth/orbbec_astra.dae"/>
+          <mesh filename="file://$(find golf_cart)/meshes/depth/orbbec_astra.stl"/>
         </geometry>
       </visual>

File: urdf/summit_xls.urdf.xacro (robot description, xacro)
@@ -34,5 +34,5 @@
 	<xacro:property name="hq" value="false" />
 	<xacro:arg name="prefix" default="summit_xl_"/>
-	<xacro:arg name="ros_planar_move_plugin" default="true"/>
+	<xacro:arg name="ros_planar_move_plugin" default="false"/>
 	<xacro:arg name="gpu" default="false"/>
     <xacro:macro name="summit_xl" params="prefix publish_bf hq">
@@ -56,10 +56,10 @@
 			<origin xyz="${front_rgbd_camera_offset_x} ${front_rgbd_camera_offset_y} ${front_rgbd_camera_offset_z}" rpy="0 0 0"/>
 		</xacro:sensor_orbbec_astra>
-		<!-- <xacro:sensor_sick_s300 frame_prefix="$(arg prefix)front_laser" parent="$(arg prefix)base_link" topic_prefix="front_laser" gpu="$(arg gpu)">
+		<xacro:sensor_sick_s300 frame_prefix="$(arg prefix)front_laser" parent="$(arg prefix)base_link" topic_prefix="front_laser" gpu="$(arg gpu)">
 			<origin xyz="${front_laser_offset_x} ${front_laser_offset_y} ${front_laser_offset_z}" rpy="0 ${-PI} ${3/4*PI}" />
 		</xacro:sensor_sick_s300>
 		<xacro:sensor_sick_s300 frame_prefix="$(arg prefix)rear_laser" parent="$(arg prefix)base_link" topic_prefix="rear_laser" gpu="$(arg gpu)">
 			<origin xyz="${rear_laser_offset_x} ${rear_laser_offset_y} ${rear_laser_offset_z}" rpy="0 ${-PI} ${-1/4*PI}" />
-		</xacro:sensor_sick_s300> -->
+		</xacro:sensor_sick_s300>
    </xacro:macro>
    <xacro:ros2_control prefix="$(arg prefix)"/>
