Commit message: detect human and get the distance between camera and human

File: urdf/summit_xls.urdf.xacro (robot description, xacro)
@@ -28,5 +28,5 @@
 	<xacro:property name="front_rgbd_camera_offset_x" value="0.35850"/>
 	<xacro:property name="front_rgbd_camera_offset_y" value="0.0"/>
-	<xacro:property name="front_rgbd_camera_offset_z" value="0.25062"/>
+	<xacro:property name="front_rgbd_camera_offset_z" value="0.8"/>
 	<xacro:property name="gps_offset_x" value="-0.365"/>
 	<xacro:property name="gps_offset_y" value="-0.167"/>

Commit message: nav2 setup

File: urdf/summit_xls.urdf.xacro (robot description, xacro)
@@ -34,20 +34,20 @@
 	<xacro:property name="hq" value="false" />
 	<xacro:arg name="prefix" default="summit_xl_"/>
-	<xacro:arg name="ros_planar_move_plugin" default="false"/>
+	<xacro:arg name="ros_planar_move_plugin" default="true"/>
 	<xacro:arg name="gpu" default="false"/>
     <xacro:macro name="summit_xl" params="prefix publish_bf hq">
 		<xacro:summit_xls_base prefix="$(arg prefix)" publish_bf="true" hq="${hq}" />
-		<xacro:rubber_wheel prefix="$(arg prefix)front_right" parent="$(arg prefix)base_link" reflect="false" hq="${hq}">
+		<xacro:omni_wheel prefix="$(arg prefix)front_right" parent="$(arg prefix)base_link" reflect="false" hq="${hq}">
 			<origin xyz="${wheel_offset_x} -${wheel_offset_y} ${wheel_offset_z}" rpy="0 0 0"/>
-		</xacro:rubber_wheel>
-		<xacro:rubber_wheel prefix="$(arg prefix)front_left" parent="$(arg prefix)base_link" reflect="true" hq="${hq}">
+		</xacro:omni_wheel>
+		<xacro:omni_wheel prefix="$(arg prefix)front_left" parent="$(arg prefix)base_link" reflect="true" hq="${hq}">
 			<origin xyz="${wheel_offset_x} ${wheel_offset_y} ${wheel_offset_z}" rpy="0 0 0"/>
-		</xacro:rubber_wheel>
-		<xacro:rubber_wheel prefix="$(arg prefix)back_left" parent="$(arg prefix)base_link" reflect="true" hq="${hq}">
+		</xacro:omni_wheel>
+		<xacro:omni_wheel prefix="$(arg prefix)back_left" parent="$(arg prefix)base_link" reflect="true" hq="${hq}">
 			<origin xyz="-${wheel_offset_x} ${wheel_offset_y} ${wheel_offset_z}" rpy="0 0 0"/>
-		</xacro:rubber_wheel>
-		<xacro:rubber_wheel prefix="$(arg prefix)back_right" parent="$(arg prefix)base_link" reflect="false" hq="${hq}">
+		</xacro:omni_wheel>
+		<xacro:omni_wheel prefix="$(arg prefix)back_right" parent="$(arg prefix)base_link" reflect="false" hq="${hq}">
 			<origin xyz="-${wheel_offset_x} -${wheel_offset_y} ${wheel_offset_z}" rpy="0 0 0"/>
-		</xacro:rubber_wheel>
+		</xacro:omni_wheel>
 		<xacro:sensor_myahrs frame_prefix="$(arg prefix)imu" parent="$(arg prefix)base_link">
 			<origin xyz="${imu_offset_x} ${imu_offset_y} ${imu_offset_z}" rpy="0 0 0"/>
@@ -65,5 +65,5 @@
    <xacro:ros2_control prefix="$(arg prefix)"/>
    <xacro:if value="$(arg ros_planar_move_plugin)">
-	   <xacro:omni_steering prefix="$(arg prefix)" publish_tf="true"/>
+	   <xacro:omni_steering prefix="$(arg prefix)" publish_tf="false"/>
    </xacro:if>
    <xacro:summit_xl prefix="$(arg prefix)" publish_bf="true" hq="${hq}"/>

File: urdf/summit_xls_base.urdf.xacro (robot description, xacro)
@@ -2,53 +2,84 @@
 <robot name="summit_xl" xmlns:xacro="http://wiki.ros.org/xacro">
   <xacro:macro name="summit_xls_base" params="prefix publish_bf hq">
-  <xacro:property name="PI" value="3.1415926535897931"/>
-  <xacro:property name="wheel_radius" value="0.127" />
-	  <xacro:if value="${publish_bf}">
-		<link name="${prefix}base_footprint">
-		  <visual>
-			  <origin xyz="0 0 0" rpy="0 0 0" />
-			  <geometry>
-				 <box size="0.001 0.001 0.001" />
-			  </geometry>
-		  </visual>
-		</link>
-		<joint name="${prefix}base_footprint_joint" type="fixed">
-		  <origin xyz="0 0 ${wheel_radius}" rpy="0 0 0" />
-		  <parent link="${prefix}base_footprint"/>
-		  <child link="${prefix}base_link" />
-		</joint>
-	  </xacro:if>
-  <link name="${prefix}base_link">
-    <inertial>
-      <mass value="125.0" />
-      <origin xyz="0 0 0" />
-      <inertia  ixx="1.391" ixy="0.004"  ixz="0.0"  iyy="6.853"  iyz="0.0"  izz="6.125" />
-    </inertial>
-    <visual>
-      <origin xyz="0 0 0" rpy="0 0 0" />
-      <xacro:if value="${hq}">
-      <geometry>
-      <mesh filename="file://$(find golf_cart)/meshes/bases/summit_xls_chassis.stl"/>
-      </geometry>
+    <xacro:property name="PI" value="3.1415926535897931"/>
+    <xacro:property name="wheel_radius" value="0.127" />
+      <xacro:if value="${publish_bf}">
+      <link name="${prefix}base_footprint">
+        <visual>
+          <origin xyz="0 0 0" rpy="0 0 0" />
+          <geometry>
+          <box size="0.001 0.001 0.001" />
+          </geometry>
+        </visual>
+      </link>
+      <joint name="${prefix}base_footprint_joint" type="fixed">
+        <origin xyz="0 0 ${wheel_radius}" rpy="0 0 0" />
+        <parent link="${prefix}base_footprint"/>
+        <child link="${prefix}base_link" />
+      </joint>
       </xacro:if>
-      <xacro:unless value="${hq}">
-      <geometry>
-      <mesh filename="file://$(find golf_cart)/meshes/bases/summit_xls_chassis.dae"/>
-      </geometry>
-      </xacro:unless>
-      <material name="white">
-        <color rgba="1.0 1.0 1.0 1"/>
-      </material>
-    </visual>
-    <collision>
-       <origin xyz="0 0 0" rpy="0 0 0 " />
-       <geometry>
-         <mesh filename="file://$(find golf_cart)/meshes/bases/summit_xls_chassis.dae"/>
-       </geometry>
-    </collision>
-  </link>
-  <gazebo reference="${prefix}base_link">
-    <material>Gazebo/Black</material>
-  </gazebo>
+    <link name="${prefix}base_link">
+      <inertial>
+        <mass value="10.0" />
+        <origin xyz="0 0 0" />
+        <inertia  ixx="1.391" ixy="0.004"  ixz="0.0"  iyy="6.853"  iyz="0.0"  izz="6.125" />
+      </inertial>
+      <visual>
+        <origin xyz="0 0 0" rpy="0 0 0" />
+        <xacro:if value="${hq}">
+        <geometry>
+        <mesh filename="file://$(find golf_cart)/meshes/bases/summit_xls_chassis.stl"/>
+        </geometry>
+        </xacro:if>
+        <xacro:unless value="${hq}">
+        <geometry>
+        <mesh filename="file://$(find golf_cart)/meshes/bases/summit_xls_chassis.dae"/>
+        </geometry>
+        </xacro:unless>
+        <material name="white">
+          <color rgba="1.0 1.0 1.0 1"/>
+        </material>
+      </visual>
+      <collision>
+        <origin xyz="0 0 0" rpy="0 0 0 " />
+        <geometry>
+          <mesh filename="file://$(find golf_cart)/meshes/bases/summit_xls_chassis.dae"/>
+        </geometry>
+      </collision>
+    </link>
+    <gazebo reference="${prefix}base_link">
+      <material>Gazebo/Black</material>
+    </gazebo>
+  </xacro:macro>
+  <xacro:macro name="omni_steering" params="prefix publish_tf force_based:=false">
+		<xacro:if value="${force_based}">
+			<gazebo>
+				<plugin name="ros_force_based_move" filename="librobotnik_force_based_move.so">
+					<commandTopic>robotnik_base_control/reference_unstamped</commandTopic>
+					<odometryTopic>odom</odometryTopic>
+					<odometryFrame>odom</odometryFrame>
+					<yaw_velocity_p_gain>10000.0</yaw_velocity_p_gain>
+					<x_velocity_p_gain>10000.0</x_velocity_p_gain>
+					<y_velocity_p_gain>10000.0</y_velocity_p_gain>
+					<robotBaseFrame>summit_xl_base_footprint</robotBaseFrame>
+					<commandWatchdog>1</commandWatchdog>
+					<odometryRate>50.0</odometryRate>
+					<publishOdometryTf>${publish_tf}</publishOdometryTf>
+				</plugin>
+			</gazebo>
+		</xacro:if>
+		<xacro:unless value="${force_based}">
+			<gazebo>
+				<plugin name="omni_steering" filename="libgazebo_ros_planar_move.so">
+				<command_topic>robotnik_base_control/reference_unstamped</command_topic>
+				<odometry_topic>odom</odometry_topic>
+				<odometry_frame>odom</odometry_frame>
+				<odometry_rate>50.0</odometry_rate>
+				<robot_base_frame>summit_xl_base_footprint</robot_base_frame>
+				<publish_tf>${publish_tf}</publish_tf>
+				<enableYAxis>true</enableYAxis>
+				</plugin>
+			</gazebo>
+		</xacro:unless>
   </xacro:macro>
 </robot>
